File: anavi-light-controller.sch (KiCad schematic (older format))
At the start: 22 parts, among them J1 Screw_Terminal_1x04, P1 CONN_01X03, Q1 IRF8721PBF-1, Q2 IRF8721PBF-1, Q3 IRF8721PBF-1, SW1 SW_DIP_x01, U1 I2C_SENS_1, U2 I2C_SENS_1, U3 I2C_SENS_1

Commit message: Updated files to kicad 5.1
Parts:
- C1, C2: symbol C -> anavi-light-controller-rescue:C
- D1: symbol LED -> anavi-light-controller-rescue:LED
- DC1: symbol dc_jack -> anavi-light-controller-rescue:dc_jack
- ESP-12: symbol ESP-12E -> anavi-light-controller-rescue:ESP-12E
- J1: symbol Screw_Terminal_1x04 -> anavi-light-controller-rescue:Screw_Terminal_1x04
- P1: symbol CONN_01X03 -> anavi-light-controller-rescue:CONN_01X03
- Q1, Q2, Q3: symbol IRF8721PBF-1 -> anavi-light-controller-rescue:IRF8721PBF-1
- R1, R2, R3, R4, R5, R6, R7: symbol R -> anavi-light-controller-rescue:R
- SW1: symbol SW_DIP_x01 -> anavi-light-controller-rescue:SW_DIP_x01
- U1, U2, U3: symbol I2C_SENS_1 -> anavi-light-controller-rescue:I2C_SENS_1
- V1: symbol LD1117S33TR -> anavi-light-controller-rescue:LD1117S33TR
